Commit message: commented out t265

File: legged_perceptive_description/urdf/robot.xacro (robot description, xacro)
@@ -6,10 +6,10 @@
     <xacro:include filename="$(find legged_perceptive_description)/urdf/sensor_t265.xacro"/>
     <xacro:include filename="$(find legged_perceptive_description)/urdf/mid360.xacro"/>
-    <!--    <xacro:sensor_d435 name="front_camera" topics_ns="front_camera" parent="base">-->
-    <!--        <origin xyz="0.36 -0.0 0.01" rpy="3.141 0.38 0"/>-->
-    <!--    </xacro:sensor_d435>-->
-    <xacro:sensor_t265 name="tracking_camera" topics_ns="tracking_camera" parent="base">
+    <xacro:sensor_d435 name="front_camera" topics_ns="front_camera" parent="base">
+        <origin xyz="0.36 -0.0 0.01" rpy="3.141 0.38 0"/>
+    </xacro:sensor_d435>
+    <!-- <xacro:sensor_t265 name="tracking_camera" topics_ns="tracking_camera" parent="base">
         <origin xyz="0.16 0 0.085" rpy="0 -1.04 0"/>
-    </xacro:sensor_t265>
+    </xacro:sensor_t265> -->
     <xacro:mid360 name="livox_right" parent="base">
         <origin xyz="0.365 -0.068 -0.030" rpy="-2.59 1.03 3.09"/>

Commit message: works in simulation now

File: legged_perceptive_description/urdf/robot.xacro (robot description, xacro)
@@ -1,16 +1,29 @@
 <?xml version="1.0"?>
 <robot xmlns:xacro="http://www.ros.org/wiki/xacro" name="robot">
-    <xacro:arg name="sim" default="false"/>
-    <xacro:include filename="$(find legged_unitree_description)/urdf/robot.xacro"/>
-    <xacro:include filename="$(find legged_perceptive_description)/urdf/sensor_d435.xacro"/>
-    <xacro:include filename="$(find legged_perceptive_description)/urdf/sensor_t265.xacro"/>
+    <xacro:arg name="sim" default="false" />
+    <xacro:include filename="$(find legged_unitree_description)/urdf/robot.xacro" />
+    <xacro:include filename="$(find legged_perceptive_description)/urdf/sensor_d435.xacro" />
+    <xacro:include filename="$(find legged_perceptive_description)/urdf/sensor_t265.xacro" />
     <!-- <xacro:include filename="$(find legged_perceptive_description)/urdf/mid360.xacro"/> -->
-    <xacro:sensor_d435 name="front_camera" topics_ns="front_camera" parent="base">
-        <origin xyz="0.36 -0.0 0.01" rpy="3.141 0.38 0"/>
+    <xacro:sensor_d435 name="depth_camera" topics_ns="depth_camera" parent="base">
+        <origin xyz="0.32 0 0.0725" rpy="0 0 0" />
+        <!-- <origin xyz="0.36 -0.0 0.01" rpy="3.141 0.38 0" /> -->
     </xacro:sensor_d435>
+    <gazebo>
+        <plugin name="base_ground_truth_pose" filename="libgazebo_ros_p3d.so">
+            <alwaysOn>true</alwaysOn>
+            <updateRate>50.0</updateRate>
+            <bodyName>base</bodyName>
+            <topicName>tracking_camera/odom/sample</topicName>
+            <gaussianNoise>0</gaussianNoise>
+            <frameName>world</frameName>
+            <xyzOffsets>0 0 0</xyzOffsets>
+            <rpyOffsets>0 0 0</rpyOffsets>
+        </plugin>
+    </gazebo>
     <!-- <xacro:sensor_t265 name="tracking_camera" topics_ns="tracking_camera" parent="base">
         <origin xyz="0.16 0 0.085" rpy="0 -1.04 0"/>
     </xacro:sensor_t265> -->
-<!--
+    <!--
     <xacro:mid360 name="livox_right" parent="base">
         <origin xyz="0.365 -0.068 -0.030" rpy="-2.59 1.03 3.09"/>

File: legged_perceptive_description/urdf/sensor_d435.xacro (robot description, xacro)
@@ -2,59 +2,62 @@
 <robot xmlns:xacro="http://ros.org/wiki/xacro">
     <xacro:macro name="sensor_d435"
-                 params="name:=camera topics_ns:=camera parent *origin publish_pointcloud:=true sim:=true">
-        <xacro:property name="M_PI" value="3.1415926535897931"/>
+        params="name:=camera topics_ns:=camera parent *origin publish_pointcloud:=true sim:=true">
+        <xacro:property name="M_PI" value="3.1415926535897931" />
         <!-- The following values are approximate, and the camera node
          publishing TF values with actual calibrated camera extrinsic values -->
-        <xacro:property name="d435_cam_depth_to_left_ir_offset" value="0.0"/>
-        <xacro:property name="d435_cam_depth_to_right_ir_offset" value="-0.050"/>
-        <xacro:property name="d435_cam_depth_to_color_offset" value="0.015"/>
+        <xacro:property name="d435_cam_depth_to_left_ir_offset" value="0.0" />
+        <xacro:property name="d435_cam_depth_to_right_ir_offset" value="-0.050" />
+        <xacro:property name="d435_cam_depth_to_color_offset" value="0.015" />
         <!-- The following values model the aluminum peripherial case for the
         D435 camera, with the camera joint represented by the actual
         peripherial camera tripod mount -->
-        <xacro:property name="d435_cam_width" value="0.090"/>
-        <xacro:property name="d435_cam_height" value="0.025"/>
-        <xacro:property name="d435_cam_depth" value="0.02505"/>
-        <xacro:property name="d435_cam_mount_from_center_offset" value="0.0149"/>
+        <xacro:property name="d435_cam_width" value="0.090" />
+        <xacro:property name="d435_cam_height" value="0.025" />
+        <xacro:property name="d435_cam_depth" value="0.02505" />
+        <xacro:property name="d435_cam_mount_from_center_offset" value="0.0149" />
         <!-- The following offset is relative the physical D435 camera peripherial
         camera tripod mount -->
-        <xacro:property name="d435_cam_depth_px" value="${d435_cam_mount_from_center_offset}"/>
-        <xacro:property name="d435_cam_depth_py" value="0.0175"/>
-        <xacro:property name="d435_cam_depth_pz" value="${d435_cam_height/2}"/>
+        <xacro:property name="d435_cam_depth_px" value="${d435_cam_mount_from_center_offset}" />
+        <xacro:property name="d435_cam_depth_py" value="0.0175" />
+        <xacro:property name="d435_cam_depth_pz" value="${d435_cam_height/2}" />
         <material name="${name}_aluminum">
-            <color rgba="0.5 0.5 0.5 1"/>
+            <color rgba="0.5 0.5 0.5 1" />
         </material>
         <!-- camera body, with origin at bottom screw mount -->
         <joint name="${name}_joint" type="fixed">
-            <xacro:insert_block name="origin"/>
-            <parent link="${parent}"/>
-            <child link="${name}_bottom_screw_frame"/>
+            <xacro:insert_block name="origin" />
+            <parent link="${parent}" />
+            <child link="${name}_bottom_screw_frame" />
         </joint>
-        <link name="${name}_bottom_screw_frame"/>
+        <link name="${name}_bottom_screw_frame" />
         <joint name="${name}_link_joint" type="fixed">
-            <origin xyz="0 ${d435_cam_depth_py} ${d435_cam_depth_pz}" rpy="0 0 0"/>
-            <parent link="${name}_bottom_screw_frame"/>
-            <child link="${name}_link"/>
+            <origin xyz="0 ${d435_cam_depth_py} ${d435_cam_depth_pz}" rpy="0 0 0" />
+            <parent link="${name}_bottom_screw_frame" />
+            <child link="${name}_link" />
         </joint>
         <link name="${name}_link">
             <visual>
-                <origin xyz="${d435_cam_mount_from_center_offset} ${-d435_cam_depth_py} 0" rpy="${M_PI/2} 0 ${M_PI/2}"/>
+                <origin xyz="${d435_cam_mount_from_center_offset} ${-d435_cam_depth_py} 0"
+                    rpy="${M_PI/2} 0 ${M_PI/2}" />
                 <geometry>
                     <!-- <box size="${d435_cam_width} ${d435_cam_height} ${d435_cam_depth}"/> -->
-                    <mesh filename="package://realsense2_description/meshes/d435.dae"/>
-                    <!--<mesh filename="package://realsense2_description/meshes/d435/d435.dae" />-->
+                    <mesh filename="package://realsense2_description/meshes/d435.dae" />
+                    <!--<mesh
+                    filename="package://realsense2_description/meshes/d435/d435.dae" />-->
                 </geometry>
-                <material name="${name}_aluminum"/>
+                <material name="${name}_aluminum" />
             </visual>
             <collision>
-                <origin xyz="0 ${-d435_cam_depth_py} 0" rpy="0 0 0"/>
+                <origin xyz="0 ${-d435_cam_depth_py} 0" rpy="0 0 0" />
                 <geometry>
-                    <box size="${d435_cam_depth} ${d435_cam_width} ${d435_cam_height}"/>
+                    <box size="${d435_cam_depth} ${d435_cam_width} ${d435_cam_height}" />
                 </geometry>
             </collision>
             <inertial>
                 <!-- The following are not reliable values, and should not be used for modeling -->
-                <mass value="0.072"/>
-                <origin xyz="0 0 0"/>
-                <inertia ixx="0.003881243" ixy="0.0" ixz="0.0" iyy="0.000498940" iyz="0.0" izz="0.003879257"/>
+                <mass value="0.072" />
+                <origin xyz="0 0 0" />
+                <inertia ixx="0.003881243" ixy="0.0" ixz="0.0" iyy="0.000498940" iyz="0.0"
+                    izz="0.003879257" />
             </inertial>
         </link>
@@ -62,62 +65,81 @@
             <!-- camera depth joints and links -->
             <joint name="${name}_depth_joint" type="fixed">
-                <origin xyz="0 0 0" rpy="0 0 0"/>
-                <parent link="${name}_link"/>
-                <child link="${name}_depth_frame"/>
+                <origin xyz="0 0 0" rpy="0 0 0" />
+                <parent link="${name}_link" />
+                <child link="${name}_depth_frame" />
             </joint>
-            <link name="${name}_depth_frame"/>
+            <link name="${name}_depth_frame" />
             <joint name="${name}_depth_optical_joint" type="fixed">
-                <origin xyz="0 0 0" rpy="${-M_PI/2} 0 ${-M_PI/2}"/>
-                <parent link="${name}_depth_frame"/>
-                <child link="${name}_depth_optical_frame"/>
+                <origin xyz="0 0 0" rpy="${-M_PI/2} 0 ${-M_PI/2}" />
+                <parent link="${name}_depth_frame" />
+                <child link="${name}_depth_optical_frame" />
             </joint>
-            <link name="${name}_depth_optical_frame"/>
+            <link name="${name}_depth_optical_frame" />
             <!-- camera left IR joints and links -->
             <joint name="${name}_left_ir_joint" type="fixed">
-                <origin xyz="0 ${d435_cam_depth_to_left_ir_offset} 0" rpy="0 0 0"/>
-                <parent link="${name}_depth_frame"/>
-                <child link="${name}_left_ir_frame"/>
+                <origin xyz="0 ${d435_cam_depth_to_left_ir_offset} 0" rpy="0 0 0" />
+                <parent link="${name}_depth_frame" />
+                <child link="${name}_left_ir_frame" />
             </joint>
-            <link name="${name}_left_ir_frame"/>
+            <link name="${name}_left_ir_frame" />
             <joint name="${name}_left_ir_optical_joint" type="fixed">
-                <origin xyz="0 0 0" rpy="${-M_PI/2} 0 ${-M_PI/2}"/>
-                <parent link="${name}_left_ir_frame"/>
-                <child link="${name}_left_ir_optical_frame"/>
+                <origin xyz="0 0 0" rpy="${-M_PI/2} 0 ${-M_PI/2}" />
+                <parent link="${name}_left_ir_frame" />
+                <child link="${name}_left_ir_optical_frame" />
             </joint>
-            <link name="${name}_left_ir_optical_frame"/>
+            <link name="${name}_left_ir_optical_frame" />
             <!-- camera right IR joints and links -->
             <joint name="${name}_right_ir_joint" type="fixed">
-                <origin xyz="0 ${d435_cam_depth_to_right_ir_offset} 0" rpy="0 0 0"/>
-                <parent link="${name}_depth_frame"/>
-                <child link="${name}_right_ir_frame"/>
+                <origin xyz="0 ${d435_cam_depth_to_right_ir_offset} 0" rpy="0 0 0" />
+                <parent link="${name}_depth_frame" />
+                <child link="${name}_right_ir_frame" />
             </joint>
-            <link name="${name}_right_ir_frame"/>
+            <link name="${name}_right_ir_frame" />
             <joint name="${name}_right_ir_optical_joint" type="fixed">
-                <origin xyz="0 0 0" rpy="${-M_PI/2} 0 ${-M_PI/2}"/>
-                <parent link="${name}_right_ir_frame"/>
-                <child link="${name}_right_ir_optical_frame"/>
+                <origin xyz="0 0 0" rpy="${-M_PI/2} 0 ${-M_PI/2}" />
+                <parent link="${name}_right_ir_frame" />
+                <child link="${name}_right_ir_optical_frame" />
             </joint>
-            <link name="${name}_right_ir_optical_frame"/>
+            <link name="${name}_right_ir_optical_frame" />
             <!-- camera color joints and links -->
             <joint name="${name}_color_joint" type="fixed">
-                <origin xyz="0 ${d435_cam_depth_to_color_offset} 0" rpy="0 0 0"/>
-                <parent link="${name}_depth_frame"/>
-                <child link="${name}_color_frame"/>
+                <origin xyz="0 ${d435_cam_depth_to_color_offset} 0" rpy="0 0 0" />
+                <parent link="${name}_depth_frame" />
+                <child link="${name}_color_frame" />
             </joint>
-            <link name="${name}_color_frame"/>
+            <link name="${name}_color_frame" />
             <joint name="${name}_color_optical_joint" type="fixed">
-                <origin xyz="0 0 0" rpy="${-M_PI/2} 0 ${-M_PI/2}"/>
-                <parent link="${name}_color_frame"/>
-                <child link="${name}_color_optical_frame"/>
+                <origin xyz="0 0 0" rpy="${-M_PI/2} 0 ${-M_PI/2}" />
+                <parent link="${name}_color_frame" />
+                <child link="${name}_color_optical_frame" />
             </joint>
-            <link name="${name}_color_optical_frame"/>
-            <xacro:include filename="$(find legged_perceptive_description)/urdf/gazebo_d400.xacro"/>
+            <link name="${name}_color_optical_frame" />
+            <!-- <gazebo reference="${name}_link_joint">
+                <disableFixedJointLumping>false</disableFixedJointLumping>
+            </gazebo> -->
+            <!-- <gazebo reference="${name}_link_joint">
+                <preserveFixedJoint>true</preserveFixedJoint>
+            </gazebo> -->
+            <!-- <gazebo>
+                <plugin name="depth_camera_ground_truth_pose" filename="libgazebo_ros_p3d.so">
+                    <alwaysOn>true</alwaysOn>
+                    <updateRate>50.0</updateRate>
+                    <bodyName>${name}_link</bodyName>
+                    <topicName>tracking_camera/odom/sample</topicName>
+                    <gaussianNoise>0</gaussianNoise>
+                    <frameName>world</frameName>
+                    <xyzOffsets>0 0 0</xyzOffsets>
+                    <rpyOffsets>0 0 0</rpyOffsets>
+                </plugin>
+            </gazebo> -->
+            <xacro:include filename="$(find legged_perceptive_description)/urdf/gazebo_d400.xacro" />
             <!-- Realsense Gazebo Plugin -->
-            <xacro:gazebo_d400 camera_name="${name}" reference_link="${name}_link" topics_ns="${topics_ns}"
-                               depth_optical_frame="${name}_depth_optical_frame"
-                               color_optical_frame="${name}_color_optical_frame"
-                               infrared1_optical_frame="${name}_left_ir_optical_frame"
-                               infrared2_optical_frame="${name}_right_ir_optical_frame"
-                               publish_pointcloud="${publish_pointcloud}"/>
+            <xacro:gazebo_d400 camera_name="${name}" reference_link="${name}_link"
+                topics_ns="${topics_ns}"
+                depth_optical_frame="${name}_depth_optical_frame"
+                color_optical_frame="${name}_color_optical_frame"
+                infrared1_optical_frame="${name}_left_ir_optical_frame"
+                infrared2_optical_frame="${name}_right_ir_optical_frame"
+                publish_pointcloud="${publish_pointcloud}" />
         </xacro:if>
     </xacro:macro>
